File: electric_project/telemetria_hardware/2020/PCB TGE2021 v1/PCB Telemetria 2020.sch (EAGLE design)
At the start: 22 parts, among them IC1 INA240A1DR, IC2 MCP3221A6T-E_OTVAO, IC3 AZ1117IH-3.3TRG1, IC4 ACS758LCB-050B-PFF-T

Commit message: XT60 changes
Parts:
- removed U$3: XT60, XT60:XT60
- added J1, J2: 74655095R, SamacSys_Parts:74655095R
Connections:
- net CMPPT_M: now also J1.1, J1.2, J1.3, J1.4, J1.5, J1.6, J1.7, J1.8; no longer U$3.-
- net CMPPT_P: now also J2.1, J2.2, J2.3, J2.4, J2.5, J2.6, J2.7, J2.8; no longer U$3.+
Changed lines of the file:
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@@
 <part name="R4" library="rcl" library_urn="urn:adsk.eagle:library:334" deviceset="R-US_" device="R0805" package3d_urn="urn:adsk.eagle:package:23553/2" value="4.7k"/>
 <part name="GND8" library="supply1" library_urn="urn:adsk.eagle:library:371" deviceset="GND" device=""/>
-<part name="U$3" library="XT60" deviceset="XT60" device=""/>
+<part name="J1" library="SamacSys_Parts" deviceset="74655095R" device=""/>
+<part name="J2" library="SamacSys_Parts" deviceset="74655095R" device=""/>
 </parts>
 <sheets>
@@
 <attribute name="VALUE" x="226.06" y="157.48" size="1.778" layer="96"/>
 </instance>
-<instance part="U$3" gate="G$1" x="203.2" y="213.36" smashed="yes" rot="R90"/>
+<instance part="J1" gate="G$1" x="170.18" y="220.98" smashed="yes">
+<attribute name="NAME" x="173.99" y="228.6" size="1.778" layer="95" align="center-left"/>
+<attribute name="VALUE" x="173.99" y="226.06" size="1.778" layer="96" align="center-left"/>
+</instance>
+<instance part="J2" gate="G$1" x="215.9" y="220.98" smashed="yes">
+<attribute name="NAME" x="219.71" y="228.6" size="1.778" layer="95" align="center-left"/>
+<attribute name="VALUE" x="219.71" y="226.06" size="1.778" layer="96" align="center-left"/>
+</instance>
 </instances>
 <busses>
@@
 <pinref part="IC4" gate="G$1" pin="IP+"/>
 <wire x1="215.9" y1="190.5" x2="220.98" y2="190.5" width="0.1524" layer="91"/>
-<label x="220.98" y="205.74" size="1.27" layer="95" xref="yes"/>
-<wire x1="220.98" y1="205.74" x2="220.98" y2="190.5" width="0.1524" layer="91"/>
-<pinref part="U$3" gate="G$1" pin="+"/>
-<wire x1="220.98" y1="205.74" x2="205.74" y2="205.74" width="0.1524" layer="91"/>
-<wire x1="205.74" y1="205.74" x2="205.74" y2="208.28" width="0.1524" layer="91"/>
+<wire x1="220.98" y1="190.5" x2="220.98" y2="195.58" width="0.1524" layer="91"/>
+<label x="220.98" y="195.58" size="1.27" layer="95" rot="R90" xref="yes"/>
+</segment>
+<segment>
+<pinref part="J2" gate="G$1" pin="1"/>
+<wire x1="215.9" y1="220.98" x2="213.36" y2="220.98" width="0.1524" layer="91"/>
+<wire x1="213.36" y1="220.98" x2="213.36" y2="218.44" width="0.1524" layer="91"/>
+<wire x1="213.36" y1="218.44" x2="213.36" y2="215.9" width="0.1524" layer="91"/>
+<wire x1="213.36" y1="208.28" x2="213.36" y2="213.36" width="0.1524" layer="91"/>
+<pinref part="J2" gate="G$1" pin="3"/>
+<wire x1="213.36" y1="213.36" x2="213.36" y2="215.9" width="0.1524" layer="91"/>
+<wire x1="215.9" y1="215.9" x2="213.36" y2="215.9" width="0.1524" layer="91"/>
+<junction x="213.36" y="215.9"/>
+<pinref part="J2" gate="G$1" pin="2"/>
+<wire x1="215.9" y1="218.44" x2="213.36" y2="218.44" width="0.1524" layer="91"/>
+<junction x="213.36" y="218.44"/>
+<pinref part="J2" gate="G$1" pin="4"/>
+<wire x1="215.9" y1="213.36" x2="213.36" y2="213.36" width="0.1524" layer="91"/>
+<junction x="213.36" y="213.36"/>
+<label x="213.36" y="208.28" size="1.27" layer="95" rot="R270" xref="yes"/>
+</segment>
+<segment>
+<pinref part="J2" gate="G$1" pin="5"/>
+<wire x1="236.22" y1="220.98" x2="238.76" y2="220.98" width="0.1524" layer="91"/>
+<wire x1="238.76" y1="220.98" x2="238.76" y2="218.44" width="0.1524" layer="91"/>
+<pinref part="J2" gate="G$1" pin="8"/>
+<wire x1="238.76" y1="218.44" x2="238.76" y2="215.9" width="0.1524" layer="91"/>
+<wire x1="238.76" y1="215.9" x2="238.76" y2="213.36" width="0.1524" layer="91"/>
+<wire x1="238.76" y1="213.36" x2="238.76" y2="208.28" width="0.1524" layer="91"/>
+<wire x1="236.22" y1="213.36" x2="238.76" y2="213.36" width="0.1524" layer="91"/>
+<junction x="238.76" y="213.36"/>
+<pinref part="J2" gate="G$1" pin="7"/>
+<wire x1="236.22" y1="215.9" x2="238.76" y2="215.9" width="0.1524" layer="91"/>
+<junction x="238.76" y="215.9"/>
+<pinref part="J2" gate="G$1" pin="6"/>
+<wire x1="236.22" y1="218.44" x2="238.76" y2="218.44" width="0.1524" layer="91"/>
+<junction x="238.76" y="218.44"/>
+<label x="238.76" y="208.28" size="1.27" layer="95" rot="R270" xref="yes"/>
 </segment>
 </net>
@@
 <pinref part="IC4" gate="G$1" pin="IP-"/>
 <wire x1="190.5" y1="190.5" x2="185.42" y2="190.5" width="0.1524" layer="91"/>
-<label x="185.42" y="205.74" size="1.27" layer="95" rot="R180" xref="yes"/>
-<pinref part="U$3" gate="G$1" pin="-"/>
-<wire x1="200.66" y1="208.28" x2="200.66" y2="205.74" width="0.1524" layer="91"/>
-<wire x1="200.66" y1="205.74" x2="185.42" y2="205.74" width="0.1524" layer="91"/>
-<wire x1="185.42" y1="205.74" x2="185.42" y2="190.5" width="0.1524" layer="91"/>
-</segment>
-</net>
+<wire x1="185.42" y1="190.5" x2="185.42" y2="195.58" width="0.1524" layer="91"/>
+<label x="185.42" y="195.58" size="1.27" layer="95" rot="R90" xref="yes"/>
+</segment>
+<segment>
+<pinref part="J1" gate="G$1" pin="1"/>
+<wire x1="170.18" y1="220.98" x2="167.64" y2="220.98" width="0.1524" layer="91"/>
+<wire x1="167.64" y1="220.98" x2="167.64" y2="218.44" width="0.1524" layer="91"/>
+<pinref part="J1" gate="G$1" pin="4"/>
+<wire x1="167.64" y1="218.44" x2="167.64" y2="215.9" width="0.1524" layer="91"/>
+<wire x1="167.64" y1="215.9" x2="167.64" y2="213.36" width="0.1524" layer="91"/>
+<wire x1="167.64" y1="213.36" x2="167.64" y2="208.28" width="0.1524" layer="91"/>
+<wire x1="170.18" y1="213.36" x2="167.64" y2="213.36" width="0.1524" layer="91"/>
+<junction x="167.64" y="213.36"/>
+<pinref part="J1" gate="G$1" pin="3"/>
+<wire x1="170.18" y1="215.9" x2="167.64" y2="215.9" width="0.1524" layer="91"/>
+<junction x="167.64" y="215.9"/>
+<pinref part="J1" gate="G$1" pin="2"/>
+<wire x1="170.18" y1="218.44" x2="167.64" y2="218.44" width="0.1524" layer="91"/>
+<junction x="167.64" y="218.44"/>
+<label x="167.64" y="208.28" size="1.27" layer="95" rot="R270" xref="yes"/>
+</segment>
+<segment>
+<pinref part="J1" gate="G$1" pin="5"/>
+<wire x1="190.5" y1="220.98" x2="193.04" y2="220.98" width="0.1524" layer="91"/>
+<wire x1="193.04" y1="220.98" x2="193.04" y2="218.44" width="0.1524" layer="91"/>
+<pinref part="J1" gate="G$1" pin="8"/>
+<wire x1="193.04" y1="218.44" x2="193.04" y2="215.9" width="0.1524" layer="91"/>
+<wire x1="193.04" y1="215.9" x2="193.04" y2="213.36" width="0.1524" layer="91"/>
+<wire x1="193.04" y1="213.36" x2="190.5" y2="213.36" width="0.1524" layer="91"/>
+<junction x="193.04" y="213.36"/>
+<pinref part="J1" gate="G$1" pin="7"/>
+<wire x1="190.5" y1="215.9" x2="193.04" y2="215.9" width="0.1524" layer="91"/>
+<junction x="193.04" y="215.9"/>
+<pinref part="J1" gate="G$1" pin="6"/>
+<wire x1="193.04" y1="218.44" x2="190.5" y2="218.44" width="0.1524" layer="91"/>
+<junction x="193.04" y="218.44"/>
+<wire x1="193.04" y1="213.36" x2="193.04" y2="208.28" width="0.1524" layer="91"/>
+<label x="193.04" y="208.28" size="1.27" layer="95" rot="R270" xref="yes"/>
+</segment>
+</net>
