File: Telemetry/2020/PCB TGE2021 v1/Projeto Principal/Versao 1_02 (eric)/PCB Telemetria 2020.brd (EAGLE design)
At the start: 160 x 100 mm, 39 parts, among them IC1 INA240A1DR, IC2 MCP3221A6T-E_OTVAO, IC3 AZ1117IH-3.3TRG1, IC4 ACS758LCB-050B-PFF-T, IC5 ADS1115IDGSR, U1 ACS712ELCTR30AT

Commit message: Atualizando para o modelo correto do Sensor Hall
Parts:
- removed U1: ACS712ELCTR30AT, ACS712ELCTR30AT:SOIC127P600X175-8N
- added U2: ACS712ELCTR-05B-T, ACS712ELCTR-05B-T:SOIC127P600X175-8N
Connections:
- net GND: now also U2.3, U2.4, U2.5; no longer U1.3, U1.4, U1.5
- net HS_FILTER: now also U2.6; no longer U1.6
- net HS_OUT: now also U2.7; no longer U1.7
- net VCC_12V: now also U2.1, U2.2; no longer U1.1, U1.2
- net VCC_3V3: now also U2.8; no longer U1.8
Changed lines of the file:
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@@
 <attribute name="VALUE" x="128.27" y="20.955" size="1.27" layer="27" rot="R270"/>
 </element>
-<element name="U1" library="ACS712ELCTR30AT" package="SOIC127P600X175-8N" value="ACS712ELCTR30AT" x="120.65" y="20.32" smashed="yes">
-<attribute name="AVAILABILITY" value="Warning" x="120.65" y="20.32" size="1.778" layer="27" display="off"/>
-<attribute name="DESCRIPTION" value=" Current Sensor 30A 1 Channel Hall Effect, Open Loop Bidirectional 8-SOIC (0.154, 3.90mm Width) " x="120.65" y="20.32" size="1.778" layer="27" display="off"/>
-<attribute name="MF" value="Allegro" x="120.65" y="20.32" size="1.778" layer="27" display="off"/>
-<attribute name="MP" value="ACS712ELCTR-30A-T" x="120.65" y="20.32" size="1.778" layer="27" display="off"/>
-<attribute name="NAME" x="116.74" y="23.022" size="1.27" layer="25"/>
-<attribute name="PACKAGE" value="SOIC-8 Allegro MicroSystems LLC" x="120.65" y="20.32" size="1.778" layer="27" display="off"/>
-<attribute name="PRICE" value="None" x="120.65" y="20.32" size="1.778" layer="27" display="off"/>
-<attribute name="VALUE" x="116.74" y="17.618" size="1.27" layer="27" align="top-left"/>
+<element name="U2" library="ACS712ELCTR-05B-T" package="SOIC127P600X175-8N" value="ACS712ELCTR-05B-T" x="119.38" y="24.13" smashed="yes" rot="R270">
+<attribute name="AVAILABILITY" value="Warning" x="119.38" y="24.13" size="1.778" layer="27" rot="R270" display="off"/>
+<attribute name="DESCRIPTION" value=" Current Sensor 5A 1 Channel Hall Effect, Open Loop Bidirectional 8-SOIC (0.154, 3.90mm Width) " x="119.38" y="24.13" size="1.778" layer="27" rot="R270" display="off"/>
+<attribute name="MF" value="Allegro MicroSystems LLC" x="119.38" y="24.13" size="1.778" layer="27" rot="R270" display="off"/>
+<attribute name="MP" value="ACS712ELCTR-05B-T" x="119.38" y="24.13" size="1.778" layer="27" rot="R270" display="off"/>
+<attribute name="NAME" x="122.082" y="28.1" size="1.27" layer="25" rot="R270"/>
+<attribute name="PACKAGE" value="SOIC-8 Allegro MicroSystems LLC" x="119.38" y="24.13" size="1.778" layer="27" rot="R270" display="off"/>
+<attribute name="PRICE" value="None" x="119.38" y="24.13" size="1.778" layer="27" rot="R270" display="off"/>
+<attribute name="PURCHASE-URL" value="https://pricing.snapeda.com/search/part/ACS712ELCTR-05B-T/?ref=eda" x="119.38" y="24.13" size="1.778" layer="27" rot="R270" display="off"/>
+<attribute name="VALUE" x="116.678" y="28.1" size="1.27" layer="27" rot="R270" align="top-left"/>
 </element>
 </elements>
@@
 <contactref element="C14" pad="2"/>
 <contactref element="C15" pad="2"/>
-<contactref element="U1" pad="5"/>
-<contactref element="U1" pad="4"/>
-<contactref element="U1" pad="3"/>
+<contactref element="U2" pad="5"/>
+<contactref element="U2" pad="3"/>
+<contactref element="U2" pad="4"/>
 <wire x1="151.13" y1="90.17" x2="146.177" y2="97.536" width="0" layer="19" extent="1-1"/>
 <wire x1="117.155" y1="74.93" x2="146.177" y2="97.536" width="0" layer="19" extent="1-1"/>
@@
 <wire x1="121.285" y1="67.371" x2="118.505" y2="71.68" width="0" layer="19" extent="1-1"/>
 <wire x1="106.553" y1="97.536" x2="117.155" y2="74.93" width="0" layer="19" extent="1-1"/>
-<wire x1="143.129" y1="27.879" x2="121.285" y2="67.371" width="0" layer="19" extent="1-1"/>
-<wire x1="145.669" y1="27.879" x2="143.129" y2="27.879" width="0" layer="19" extent="1-1"/>
-<wire x1="144.592" y1="25.019" x2="145.669" y2="27.879" width="0" layer="19" extent="1-1"/>
-<wire x1="148.61" y1="29.21" x2="145.669" y2="27.879" width="0" layer="19" extent="1-1"/>
-<wire x1="145.542" y1="19.878" x2="144.592" y2="25.019" width="0" layer="19" extent="1-1"/>
-<wire x1="143.002" y1="19.878" x2="145.542" y2="19.878" width="0" layer="19" extent="1-1"/>
-<wire x1="148.419" y1="20.32" x2="145.542" y2="19.878" width="0" layer="19" extent="1-1"/>
-<wire x1="153.841" y1="20.32" x2="148.419" y2="20.32" width="0" layer="19" extent="1-1"/>
-<wire x1="130.81" y1="10.48" x2="143.002" y2="19.878" width="0" layer="19" extent="1-1"/>
-<wire x1="123.125" y1="18.415" x2="130.81" y2="10.48" width="0" layer="19" extent="1-1"/>
-<wire x1="118.175" y1="18.415" x2="123.125" y2="18.415" width="0" layer="19" extent="1-1"/>
-<wire x1="118.175" y1="19.685" x2="118.175" y2="18.415" width="0" layer="19" extent="1-1"/>
-<wire x1="110.49" y1="18.1" x2="118.175" y2="18.415" width="0" layer="19" extent="1-1"/>
+<wire x1="118.745" y1="26.605" x2="121.285" y2="67.371" width="0" layer="19" extent="1-1"/>
+<wire x1="117.475" y1="26.605" x2="118.745" y2="26.605" width="0" layer="19" extent="1-1"/>
+<wire x1="117.475" y1="21.655" x2="117.475" y2="26.605" width="0" layer="19" extent="1-1"/>
+<wire x1="110.49" y1="18.1" x2="117.475" y2="21.655" width="0" layer="19" extent="1-1"/>
 <wire x1="110.17" y1="8.89" x2="110.49" y2="18.1" width="0" layer="19" extent="1-1"/>
 <wire x1="110.17" y1="2.54" x2="110.17" y2="8.89" width="0" layer="19" extent="1-1"/>
+<wire x1="130.81" y1="10.48" x2="117.475" y2="21.655" width="0" layer="19" extent="1-1"/>
+<wire x1="143.002" y1="19.878" x2="130.81" y2="10.48" width="0" layer="19" extent="1-1"/>
+<wire x1="145.542" y1="19.878" x2="143.002" y2="19.878" width="0" layer="19" extent="1-1"/>
+<wire x1="148.419" y1="20.32" x2="145.542" y2="19.878" width="0" layer="19" extent="1-1"/>
+<wire x1="144.592" y1="25.019" x2="145.542" y2="19.878" width="0" layer="19" extent="1-1"/>
+<wire x1="145.669" y1="27.879" x2="144.592" y2="25.019" width="0" layer="19" extent="1-1"/>
+<wire x1="143.129" y1="27.879" x2="145.669" y2="27.879" width="0" layer="19" extent="1-1"/>
+<wire x1="148.61" y1="29.21" x2="145.669" y2="27.879" width="0" layer="19" extent="1-1"/>
+<wire x1="153.841" y1="20.32" x2="148.419" y2="20.32" width="0" layer="19" extent="1-1"/>
 <wire x1="49.05" y1="87.59" x2="106.553" y2="97.536" width="0" layer="19" extent="1-1"/>
 <wire x1="49.85" y1="76.2" x2="49.05" y2="87.59" width="0" layer="19" extent="1-1"/>
@@
 <contactref element="IC5" pad="8"/>
 <contactref element="C10" pad="1"/>
-<contactref element="U1" pad="8"/>
+<contactref element="U2" pad="8"/>
 <wire x1="153.67" y1="31.43" x2="156.21" y2="31.43" width="0" layer="19" extent="1-1"/>
 <wire x1="148.61" y1="30.16" x2="153.67" y2="31.43" width="0" layer="19" extent="1-1"/>
@@
 <wire x1="148.419" y1="21.59" x2="145.542" y2="21.778" width="0" layer="19" extent="1-1"/>
 <wire x1="153.841" y1="21.59" x2="148.419" y2="21.59" width="0" layer="19" extent="1-1"/>
-<wire x1="123.125" y1="22.225" x2="143.002" y2="21.778" width="0" layer="19" extent="1-1"/>
+<wire x1="121.285" y1="21.655" x2="143.002" y2="21.778" width="0" layer="19" extent="1-1"/>
 <wire x1="121.285" y1="65.471" x2="143.129" y2="29.779" width="0" layer="19" extent="1-1"/>
 <wire x1="116.205" y1="65.48" x2="121.285" y2="65.471" width="0" layer="19" extent="1-1"/>
@@
 <contactref element="12V_POWER" pad="2"/>
 <contactref element="R9" pad="1"/>
-<contactref element="U1" pad="1"/>
-<contactref element="U1" pad="2"/>
+<contactref element="U2" pad="1"/>
+<contactref element="U2" pad="2"/>
 <wire x1="146.177" y1="80.264" x2="151.13" y2="87.17" width="0" layer="19" extent="1-1"/>
-<wire x1="118.175" y1="22.225" x2="146.177" y2="80.264" width="0" layer="19" extent="1-1"/>
-<wire x1="118.175" y1="20.955" x2="118.175" y2="22.225" width="0" layer="19" extent="1-1"/>
-<wire x1="119.06" y1="8.89" x2="118.175" y2="20.955" width="0" layer="19" extent="1-1"/>
+<wire x1="121.285" y1="26.605" x2="146.177" y2="80.264" width="0" layer="19" extent="1-1"/>
+<wire x1="120.015" y1="26.605" x2="121.285" y2="26.605" width="0" layer="19" extent="1-1"/>
+<wire x1="119.06" y1="8.89" x2="120.015" y2="26.605" width="0" layer="19" extent="1-1"/>
 </signal>
 <signal name="VCC_5V">
@@
 <signal name="HS_OUT">
 <contactref element="R15" pad="1"/>
-<contactref element="U1" pad="7"/>
-<wire x1="123.125" y1="20.955" x2="130.81" y2="21.27" width="0" layer="19" extent="1-1"/>
+<contactref element="U2" pad="7"/>
+<wire x1="120.015" y1="21.655" x2="130.81" y2="21.27" width="0" layer="19" extent="1-1"/>
 </signal>
 <signal name="HS_FILTER">
 <contactref element="C14" pad="1"/>
-<contactref element="U1" pad="6"/>
-<wire x1="110.49" y1="20" x2="123.125" y2="19.685" width="0" layer="19" extent="1-1"/>
+<contactref element="U2" pad="6"/>
+<wire x1="110.49" y1="20" x2="118.745" y2="21.655" width="0" layer="19" extent="1-1"/>
 </signal>
 </signals>
