File: Telemetry/2020/PCB TGE2021 v1/Projeto Principal/Versao 1_05 (eric - editando)/PCB Telemetria 2020.brd (EAGLE design)
At the start: 160 x 100 mm, 49 parts, among them IC1 INA240A1DR, IC2 MCP3221A6T-E_OTVAO, IC3 AZ1117IH-3.3TRG1, IC4 ACS758LCB-050B-PFF-T, IC5 ADS1115IDGSR, IC6 ACS712-030B3, IC7 THVD2410DR, J1 172042-0406

Commit message: Adding temperature sensor TMP100
Parts:
- added C17: 10nF, rcl:C0805
- added R17, R18: 5k, rcl:R0805
- added U1: TMP100NA/3K, TMP100NA_3K:SOT95P280X145-6N
Connections:
- net GND: now also C17.2, U1.2, U1.3, U1.5
- net I2C_SCL: now also R17.2, U1.1
- net I2C_SDA: now also R18.1, U1.6
- net VCC_3V3: now also C17.1, R17.1, R18.2, U1.4
Changed lines of the file:
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@@
 <?xml version="1.0" encoding="utf-8"?>
 <!DOCTYPE eagle SYSTEM "eagle.dtd">
-<eagle version="9.5.2">
+<eagle version="9.6.2">
 <drawing>
 <settings>
@@
 </layers>
 <board>
-<fusionsync huburn="a.cGVyc29uYWw6dWUyZDkwMWJh" projecturn="a.cGVyc29uYWw6dWUyZDkwMWJhIzIwMjAwODE2MzIzOTA5MTA2" f3durn="urn:adsk.wipprod:dm.lineage:uE01plevSWODFXVH0NNS5w" pcbguid="52094770-dfe4-426a-9aa2-8b08af3b6d69" lastpulledtime="" lastsyncedchangeguid="81b568d7-5ed1-2049-b759-ae446f31c16f"/>
+<fusionsync huburn="a.cGVyc29uYWw6dWUyZDkwMWJh" projecturn="a.cGVyc29uYWw6dWUyZDkwMWJhIzIwMjAwODE2MzIzOTA5MTA2" f3durn="urn:adsk.wipprod:dm.lineage:uE01plevSWODFXVH0NNS5w" pcbguid="52094770-dfe4-426a-9aa2-8b08af3b6d69" lastpulledtime="" lastsyncedchangeguid="81b568d7-5ed1-2049-b759-ae446f31c16f" latestrevisionid="" lastsyncedrevisionid="" lastboardhashguid="" lastpushedtime="" linktopcb3d="false"/>
 <plain>
 <wire x1="0" y1="0" x2="160" y2="0" width="0" layer="20"/>
@@
 <attribute name="VALUE" x="2.54" y="40.64" size="1.27" layer="27" rot="R270"/>
 </element>
+<element name="U1" library="TMP100NA_3K" package="SOT95P280X145-6N" value="TMP100NA/3K" x="27.305" y="44.45" smashed="yes" rot="R270">
+<attribute name="AVAILABILITY" value="Good" x="27.305" y="44.45" size="1.778" layer="27" rot="R270" display="off"/>
+<attribute name="DESCRIPTION" value=" Temperature Sensor with I2C/SMBus Interface in SOT-23 6-SOT-23 -55 to 125 " x="27.305" y="44.45" size="1.778" layer="27" rot="R270" display="off"/>
+<attribute name="MF" value="Texas Instruments" x="27.305" y="44.45" size="1.778" layer="27" rot="R270" display="off"/>
+<attribute name="MP" value="TMP100NA/3K" x="27.305" y="44.45" size="1.778" layer="27" rot="R270" display="off"/>
+<attribute name="NAME" x="29.305" y="47.25" size="1.27" layer="25" rot="R270"/>
+<attribute name="PACKAGE" value="SOT-23-6 Texas Instruments" x="27.305" y="44.45" size="1.778" layer="27" rot="R270" display="off"/>
+<attribute name="PRICE" value="None" x="27.305" y="44.45" size="1.778" layer="27" rot="R270" display="off"/>
+<attribute name="PURCHASE-URL" value="https://pricing.snapeda.com/search/part/TMP100NA/3K/?ref=eda" x="27.305" y="44.45" size="1.778" layer="27" rot="R270" display="off"/>
+<attribute name="VALUE" x="24.305" y="47.35" size="1.27" layer="27" rot="R270"/>
+</element>
+<element name="R17" library="rcl" library_urn="urn:adsk.eagle:library:334" package="R0805" package3d_urn="urn:adsk.eagle:package:23553/2" value="5k" x="37.465" y="44.45" smashed="yes" rot="R90">
+<attribute name="NAME" x="36.195" y="43.815" size="1.27" layer="25" rot="R90"/>
+<attribute name="POPULARITY" value="85" x="37.465" y="44.45" size="1.778" layer="27" rot="R90" display="off"/>
+<attribute name="SPICEPREFIX" value="R" x="37.465" y="44.45" size="1.778" layer="27" rot="R90" display="off"/>
+<attribute name="VALUE" x="40.005" y="43.815" size="1.27" layer="27" rot="R90"/>
+</element>
+<element name="R18" library="rcl" library_urn="urn:adsk.eagle:library:334" package="R0805" package3d_urn="urn:adsk.eagle:package:23553/2" value="5k" x="45.085" y="44.45" smashed="yes" rot="R270">
+<attribute name="NAME" x="46.355" y="45.085" size="1.27" layer="25" rot="R270"/>
+<attribute name="POPULARITY" value="85" x="45.085" y="44.45" size="1.778" layer="27" rot="R270" display="off"/>
+<attribute name="SPICEPREFIX" value="R" x="45.085" y="44.45" size="1.778" layer="27" rot="R270" display="off"/>
+<attribute name="VALUE" x="42.545" y="45.085" size="1.27" layer="27" rot="R270"/>
+</element>
+<element name="C17" library="rcl" library_urn="urn:adsk.eagle:library:334" package="C0805" package3d_urn="urn:adsk.eagle:package:23617/2" value="10nF" x="53.34" y="43.815" smashed="yes">
+<attribute name="NAME" x="52.07" y="45.085" size="1.27" layer="25"/>
+<attribute name="POPULARITY" value="63" x="53.34" y="43.815" size="1.778" layer="27" display="off"/>
+<attribute name="SPICEPREFIX" value="C" x="53.34" y="43.815" size="1.778" layer="27" display="off"/>
+<attribute name="VALUE" x="52.07" y="41.275" size="1.27" layer="27"/>
+</element>
 </elements>
 <signals>
@@
 <contactref element="C16" pad="2"/>
 <contactref element="RJ11_1" pad="P$3"/>
+<contactref element="U1" pad="5"/>
+<contactref element="U1" pad="3"/>
+<contactref element="U1" pad="2"/>
+<contactref element="C17" pad="2"/>
 <wire x1="139.7" y1="48.089" x2="139.7" y2="53.511" width="0" layer="19" extent="1-1"/>
 <wire x1="140.142" y1="45.212" x2="139.7" y2="48.089" width="0" layer="19" extent="1-1"/>
@@
 <wire x1="42.352" y1="58.801" x2="49.022" y2="56.835" width="0" layer="19" extent="1-1"/>
 <wire x1="42.291" y1="61.404" x2="42.352" y2="58.801" width="0" layer="19" extent="1-1"/>
-<wire x1="2.54" y1="66.82" x2="42.291" y2="61.404" width="0" layer="19" extent="1-1"/>
-<wire x1="12.065" y1="64.775" x2="2.54" y2="66.82" width="0" layer="19" extent="1-1"/>
+<wire x1="54.29" y1="43.815" x2="62.23" y2="57.47" width="0" layer="19" extent="1-1"/>
+<wire x1="27.305" y1="45.705" x2="42.352" y2="58.801" width="0" layer="19" extent="1-1"/>
+<wire x1="26.355" y1="45.705" x2="27.305" y2="45.705" width="0" layer="19" extent="1-1"/>
+<wire x1="27.305" y1="43.195" x2="27.305" y2="45.705" width="0" layer="19" extent="1-1"/>
+<wire x1="15.24" y1="47.305" x2="26.355" y2="45.705" width="0" layer="19" extent="1-1"/>
+<wire x1="5.544" y1="46.355" x2="15.24" y2="47.305" width="0" layer="19" extent="1-1"/>
+<wire x1="5.08" y1="38.42" x2="5.544" y2="46.355" width="0" layer="19" extent="1-1"/>
+<wire x1="22.2" y1="30.95" x2="27.305" y2="43.195" width="0" layer="19" extent="1-1"/>
+<wire x1="12.065" y1="64.775" x2="15.24" y2="47.305" width="0" layer="19" extent="1-1"/>
 <wire x1="20.32" y1="66.82" x2="12.065" y2="64.775" width="0" layer="19" extent="1-1"/>
-<wire x1="5.544" y1="46.355" x2="20.32" y2="66.82" width="0" layer="19" extent="1-1"/>
-<wire x1="5.08" y1="38.42" x2="5.544" y2="46.355" width="0" layer="19" extent="1-1"/>
-<wire x1="15.24" y1="47.305" x2="5.544" y2="46.355" width="0" layer="19" extent="1-1"/>
-<wire x1="22.2" y1="30.95" x2="15.24" y2="47.305" width="0" layer="19" extent="1-1"/>
+<wire x1="2.54" y1="66.82" x2="12.065" y2="64.775" width="0" layer="19" extent="1-1"/>
 <wire x1="37.8" y1="6.05" x2="22.2" y2="30.95" width="0" layer="19" extent="1-1"/>
 </signal>
@@
 <wire x1="5.08" y1="40.32" x2="5.08" y2="42.081" width="0.508" layer="1"/>
 <wire x1="5.08" y1="42.081" x2="5.544" y2="42.545" width="0.508" layer="1"/>
+<contactref element="R18" pad="2"/>
+<contactref element="C17" pad="1"/>
+<contactref element="R17" pad="1"/>
+<contactref element="U1" pad="4"/>
 <wire x1="138.43" y1="48.089" x2="138.43" y2="53.511" width="0" layer="19" extent="1-1"/>
 <wire x1="138.242" y1="45.212" x2="138.43" y2="48.089" width="0" layer="19" extent="1-1"/>
@@
 <wire x1="62.23" y1="59.37" x2="92.785" y2="51.435" width="0" layer="19" extent="1-1"/>
 <wire x1="62.23" y1="62.57" x2="62.23" y2="59.37" width="0" layer="19" extent="1-1"/>
-<wire x1="40.452" y1="58.801" x2="62.23" y2="59.37" width="0" layer="19" extent="1-1"/>
-<wire x1="40.381" y1="61.404" x2="40.452" y2="58.801" width="0" layer="19" extent="1-1"/>
-<wire x1="35.2" y1="30.95" x2="40.452" y2="58.801" width="0" layer="19" extent="1-1"/>
+<wire x1="52.39" y1="43.815" x2="62.23" y2="59.37" width="0" layer="19" extent="1-1"/>
+<wire x1="45.085" y1="43.5" x2="52.39" y2="43.815" width="0" layer="19" extent="1-1"/>
+<wire x1="37.465" y1="43.5" x2="45.085" y2="43.5" width="0" layer="19" extent="1-1"/>
+<wire x1="35.2" y1="30.95" x2="37.465" y2="43.5" width="0" layer="19" extent="1-1"/>
 <wire x1="24.8" y1="30.95" x2="35.2" y2="30.95" width="0" layer="19" extent="1-1"/>
-<wire x1="15.875" y1="40.325" x2="24.8" y2="30.95" width="0" layer="19" extent="1-1"/>
+<wire x1="26.355" y1="43.195" x2="37.465" y2="43.5" width="0" layer="19" extent="1-1"/>
+<wire x1="15.875" y1="40.325" x2="26.355" y2="43.195" width="0" layer="19" extent="1-1"/>
 <wire x1="11.43" y1="38.42" x2="15.875" y2="40.325" width="0" layer="19" extent="1-1"/>
 <wire x1="5.08" y1="40.32" x2="11.43" y2="38.42" width="0" layer="19" extent="1-1"/>
+<wire x1="40.452" y1="58.801" x2="37.465" y2="43.5" width="0" layer="19" extent="1-1"/>
+<wire x1="40.381" y1="61.404" x2="40.452" y2="58.801" width="0" layer="19" extent="1-1"/>
 <wire x1="9.525" y1="64.775" x2="5.544" y2="42.545" width="0" layer="19" extent="1-1"/>
 </signal>
@@
 <contactref element="R1" pad="1"/>
 <contactref element="IC5" pad="9"/>
+<contactref element="R18" pad="1"/>
+<contactref element="U1" pad="6"/>
 <wire x1="130.49" y1="50.78" x2="130.49" y2="55.88" width="0" layer="19" extent="1-1"/>
-<wire x1="30" y1="30.95" x2="130.49" y2="50.78" width="0" layer="19" extent="1-1"/>
-<wire x1="62.73" y1="62.57" x2="30" y2="30.95" width="0" layer="19" extent="1-1"/>
+<wire x1="62.73" y1="62.57" x2="130.49" y2="55.88" width="0" layer="19" extent="1-1"/>
+<wire x1="45.085" y1="45.4" x2="62.73" y2="62.57" width="0" layer="19" extent="1-1"/>
+<wire x1="28.255" y1="43.195" x2="45.085" y2="45.4" width="0" layer="19" extent="1-1"/>
+<wire x1="30" y1="30.95" x2="28.255" y2="43.195" width="0" layer="19" extent="1-1"/>
 </signal>
 <signal name="I2C_SCL">
@@
 <contactref element="R2" pad="1"/>
 <contactref element="IC5" pad="10"/>
+<contactref element="R17" pad="2"/>
+<contactref element="U1" pad="1"/>
 <wire x1="128.59" y1="50.78" x2="130.49" y2="53.34" width="0" layer="19" extent="1-1"/>
-<wire x1="32.6" y1="30.95" x2="128.59" y2="50.78" width="0" layer="19" extent="1-1"/>
-<wire x1="63.23" y1="62.57" x2="32.6" y2="30.95" width="0" layer="19" extent="1-1"/>
+<wire x1="63.23" y1="62.57" x2="128.59" y2="50.78" width="0" layer="19" extent="1-1"/>
+<wire x1="37.465" y1="45.4" x2="63.23" y2="62.57" width="0" layer="19" extent="1-1"/>
+<wire x1="28.255" y1="45.705" x2="37.465" y2="45.4" width="0" layer="19" extent="1-1"/>
+<wire x1="32.6" y1="30.95" x2="37.465" y2="45.4" width="0" layer="19" extent="1-1"/>
 </signal>
 <signal name="N$27">
