File: Telemetry/2020/PCB TGE2021 v1/Projeto Principal/Versao 1_07_02 (agricio)/PCB Telemetria 2020.brd (EAGLE design)
At the start: 160 x 75.2 mm, 57 parts, among them IC1 INA240A1DR, IC2 MCP3221A6T-E_OTVAO, IC3 AZ1117IH-3.3TRG1, IC4 ACS758LCB-050B-PFF-T, IC5 ADS1115IDGSR, IC6 ACS712-030B3, IC7 THVD2410DR, IC8 TMP235AEDCKRQ1, J1 172042-0406, J2 43045-0412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

Commit message: adicionando novo conector
Parts:
- added RJ11_2: TFC44, Painel-Facilidades:TFC44
- moved D1 18.5 mm to (20.3, 69.8)
- moved C17 13.0 mm to (36.8, 39.4), turned to 180 degrees
- moved R17 12.6 mm to (36.8, 47.0), turned to 180 degrees
- moved IC8 9.52 mm to (36.8, 43.8), turned to 180 degrees
- moved C18 7.10 mm to (28.6, 43.2), turned to 270 degrees
- moved R8 5.68 mm to (65.4, 52.1)
- moved R9 4.49 mm to (98.4, 18.4)
- moved R7 3.18 mm to (70.9, 52.1)
- moved BBANK 2.69 mm to (84.5, 63.5)
- moved C7 2.69 mm to (100.3, 49.5)
- moved IC3 2.69 mm to (94.0, 49.5)
- moved R6 2.69 mm to (84.5, 48.3)
- moved VPV 2.69 mm to (69.2, 63.5)
- moved C11 2.69 mm to (84.5, 44.5)
- moved C6 2.69 mm to (91.8, 44.5)
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Connections:
- net ADC1_4 renamed 12V_VM
- net ADC1_5 renamed 12V_CM
- removed net N$12: U$1.13
- removed net TMP_ADC2_8: C18.1, R17.2, U$1.14
- new net N$4: U$1.14
- new net TEMP1: C18.1, R17.2, U$1.13
- net GND: now also RJ11_2.P$3
- net N$14: now also RJ11_2.P$4
- net N$9: now also RJ11_2.P$2
- net VCC_3V3: now also RJ11_2.P$1
Routing:
- net N$14: track 22.2 -> 44.8 mm
- net N$9: track 28.5 -> 42.4 mm
- net UART_RX: track 13.4 -> 14.9 mm
- net UART_TX: track 16.5 -> 17.8 mm
- net !RXEN: track 17.2 -> 18.4 mm
- net TXEN: track 21.1 -> 22.1 mm
