File: Telemetry/2020/PCB TGE2021 v1/Projeto Principal/Versao 1_07_02 (agricio)/PCB Telemetria 2020.sch (EAGLE design)
At the start: 57 parts, among them IC1 INA240A1DR, IC2 MCP3221A6T-E_OTVAO, IC3 AZ1117IH-3.3TRG1, IC4 ACS758LCB-050B-PFF-T, IC5 ADS1115IDGSR, IC6 ACS712-030B3, IC7 THVD2410DR, IC8 TMP235AEDCKRQ1, J1 172042-0406, J2 43045-0412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

Commit message: adicionando novo conector
Parts:
- added RJ11_2: TFC44, Painel-Facilidades:TFC44
Connections:
- net ADC1_4 renamed 12V_VM
- net ADC1_5 renamed 12V_CM
- removed net N$12: U$1.13
- removed net TMP_ADC2_8: C18.1, R17.2, U$1.14
- new net N$4: U$1.14
- new net TEMP1: C18.1, R17.2, U$1.13
- net GND: now also RJ11_2.3
- net N$14: now also RJ11_2.4
- net N$9: now also RJ11_2.2
- net VCC_3V3: now also RJ11_2.1
Other:
- moved on the sheet: BBANK, C10, C11, C12, C13, C14, C15, C17, C18, IC5, IC6, IC8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
