File: Telemetry/2020/PCB TGE2021 v1/Projeto Principal/Versao 1_07 (eric)/PCB Telemetria 2020.brd (EAGLE design)
At the start: 160 x 75.2 mm, 58 parts, among them IC1 INA240A1DR, IC2 MCP3221A6T-E_OTVAO, IC3 AZ1117IH-3.3TRG1, IC4 ACS758LCB-050B-PFF-T, IC5 ADS1115IDGSR, IC6 ACS712-030B3, IC7 THVD2410DR, IC8 TMP235AEDCKRQ1, J1 172042-0406, J2 43045-0412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

Commit message: Final v1.07
Final version with extra connectors and temperature sensor wired properly
Connections:
- removed net N$14: D2.1, IC7.7, R14.2, RJ11_1.P$4, RJ11_2.P$4
- removed net N$9: D1.1, IC7.6, R14.1, RJ11_1.P$2, RJ11_2.P$2
- new net RS485_A: D1.1, IC7.6, J5.3, R14.1, RJ11_1.P$2, RJ11_2.P$2
- new net RS485_B: D2.1, IC7.7, J5.4, R14.2, RJ11_1.P$4, RJ11_2.P$4
- net CONEX_11: now also J2.3
- net CONEX_12: now also J2.4
- net CONEX_21: now also J3.3
- net CONEX_22: now also J3.4
- net CONEX_31: now also J4.3
- net CONEX_32: now also J4.4
- net GND: now also J2.2, J3.2, J4.2, J5.2
- net VCC_5V: now also J2.1, J3.1, J4.1, J5.1
Routing:
- net RS485_B: track 0.00 -> 44.8 mm
- net N$14: track 44.8 -> 0.00 mm
- net RS485_A: track 0.00 -> 42.4 mm
- net N$9: track 42.4 -> 0.00 mm
Changed lines of the file:
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@@
 <?xml version="1.0" encoding="utf-8"?>
 <!DOCTYPE eagle SYSTEM "eagle.dtd">
-<eagle version="9.5.2">
+<eagle version="9.6.2">
 <drawing>
 <settings>
@@
 </layers>
 <board>
-<fusionsync huburn="a.cGVyc29uYWw6dWUyZDkwMWJh" projecturn="a.cGVyc29uYWw6dWUyZDkwMWJhIzIwMjAwODE2MzIzOTA5MTA2" f3durn="urn:adsk.wipprod:dm.lineage:uE01plevSWODFXVH0NNS5w" pcbguid="52094770-dfe4-426a-9aa2-8b08af3b6d69" lastpulledtime="" lastsyncedchangeguid="81b568d7-5ed1-2049-b759-ae446f31c16f"/>
+<fusionsync huburn="a.cGVyc29uYWw6dWUyZDkwMWJh" projecturn="a.cGVyc29uYWw6dWUyZDkwMWJhIzIwMjAwODE2MzIzOTA5MTA2" f3durn="urn:adsk.wipprod:dm.lineage:uE01plevSWODFXVH0NNS5w" pcbguid="52094770-dfe4-426a-9aa2-8b08af3b6d69" lastpulledtime="" lastsyncedchangeguid="81b568d7-5ed1-2049-b759-ae446f31c16f" latestrevisionid="" lastsyncedrevisionid="" lastboardhashguid="" lastpushedtime="" linktopcb3d="false"/>
 <plain>
 <wire x1="0" y1="0" x2="160" y2="0" width="0" layer="20"/>
@@
 <contactref element="C18" pad="2"/>
 <contactref element="RJ11_2" pad="P$3"/>
+<contactref element="J2" pad="2"/>
+<contactref element="J3" pad="2"/>
+<contactref element="J4" pad="2"/>
+<contactref element="J5" pad="2"/>
 <wire x1="139.7" y1="48.089" x2="139.7" y2="53.511" width="0" layer="19" extent="1-1"/>
 <wire x1="140.142" y1="45.212" x2="139.7" y2="48.089" width="0" layer="19" extent="1-1"/>
@@
 <wire x1="136.465" y1="20.955" x2="151.595" y2="32.273" width="0" layer="19" extent="1-1"/>
 <wire x1="136.525" y1="13.02" x2="136.465" y2="20.955" width="0" layer="19" extent="1-1"/>
+<wire x1="132.865" y1="4.375" x2="136.525" y2="13.02" width="0" layer="19" extent="1-1"/>
 <wire x1="127" y1="20.635" x2="136.465" y2="20.955" width="0" layer="19" extent="1-1"/>
 <wire x1="122.936" y1="16.383" x2="127" y2="20.635" width="0" layer="19" extent="1-1"/>
-<wire x1="100.33" y1="48.58" x2="122.936" y2="56.007" width="0" layer="19" extent="1-1"/>
-<wire x1="97.08" y1="47.23" x2="100.33" y2="48.58" width="0" layer="19" extent="1-1"/>
-<wire x1="92.771" y1="44.45" x2="97.08" y2="47.23" width="0" layer="19" extent="1-1"/>
+<wire x1="144.93" y1="4.375" x2="136.525" y2="13.02" width="0" layer="19" extent="1-1"/>
+<wire x1="120.8" y1="4.375" x2="132.865" y2="4.375" width="0" layer="19" extent="1-1"/>
+<wire x1="108.735" y1="4.375" x2="120.8" y2="4.375" width="0" layer="19" extent="1-1"/>
+<wire x1="97.155" y1="23.81" x2="108.735" y2="4.375" width="0" layer="19" extent="1-1"/>
+<wire x1="92.71" y1="23.81" x2="97.155" y2="23.81" width="0" layer="19" extent="1-1"/>
+<wire x1="92.771" y1="44.45" x2="92.71" y2="23.81" width="0" layer="19" extent="1-1"/>
+<wire x1="97.08" y1="47.23" x2="92.771" y2="44.45" width="0" layer="19" extent="1-1"/>
+<wire x1="100.33" y1="48.58" x2="97.08" y2="47.23" width="0" layer="19" extent="1-1"/>
 <wire x1="83.505" y1="44.45" x2="92.771" y2="44.45" width="0" layer="19" extent="1-1"/>
 <wire x1="83.505" y1="48.26" x2="83.505" y2="44.45" width="0" layer="19" extent="1-1"/>
@@
 <wire x1="67.465" y1="59.65" x2="82.705" y2="59.65" width="0" layer="19" extent="1-1"/>
 <wire x1="65.405" y1="53.02" x2="67.465" y2="59.65" width="0" layer="19" extent="1-1"/>
-<wire x1="65.405" y1="53.02" x2="67.625" y2="43.815" width="0" layer="19" extent="1-1"/>
+<wire x1="67.625" y1="43.815" x2="65.405" y2="53.02" width="0" layer="19" extent="1-1"/>
 <wire x1="67.675" y1="40.935" x2="67.625" y2="43.815" width="0" layer="19" extent="1-1"/>
 <wire x1="66.675" y1="40.935" x2="67.675" y2="40.935" width="0" layer="19" extent="1-1"/>
@@
 <wire x1="48.702" y1="31.496" x2="55.372" y2="29.53" width="0" layer="19" extent="1-1"/>
 <wire x1="48.641" y1="34.099" x2="48.702" y2="31.496" width="0" layer="19" extent="1-1"/>
-<wire x1="28.575" y1="42.23" x2="48.641" y2="34.099" width="0" layer="19" extent="1-1"/>
-<wire x1="35.88" y1="39.37" x2="28.575" y2="42.23" width="0" layer="19" extent="1-1"/>
+<wire x1="35.88" y1="39.37" x2="48.641" y2="34.099" width="0" layer="19" extent="1-1"/>
 <wire x1="37.78" y1="43.815" x2="35.88" y2="39.37" width="0" layer="19" extent="1-1"/>
-<wire x1="13.462" y1="47.686" x2="37.78" y2="43.815" width="0" layer="19" extent="1-1"/>
+<wire x1="28.575" y1="42.23" x2="35.88" y2="39.37" width="0" layer="19" extent="1-1"/>
+<wire x1="21.565" y1="30.315" x2="28.575" y2="42.23" width="0" layer="19" extent="1-1"/>
+<wire x1="13.462" y1="47.686" x2="28.575" y2="42.23" width="0" layer="19" extent="1-1"/>
 <wire x1="4.909" y1="46.99" x2="13.462" y2="47.686" width="0" layer="19" extent="1-1"/>
 <wire x1="4.445" y1="39.055" x2="4.909" y2="46.99" width="0" layer="19" extent="1-1"/>
-<wire x1="21.565" y1="30.315" x2="37.78" y2="43.815" width="0" layer="19" extent="1-1"/>
-<wire x1="29.845" y1="67.315" x2="35.88" y2="39.37" width="0" layer="19" extent="1-1"/>
-<wire x1="20.32" y1="64.915" x2="29.845" y2="67.315" width="0" layer="19" extent="1-1"/>
+<wire x1="20.32" y1="64.915" x2="13.462" y2="47.686" width="0" layer="19" extent="1-1"/>
+<wire x1="20.32" y1="71.9" x2="20.32" y2="64.915" width="0" layer="19" extent="1-1"/>
 <wire x1="12.065" y1="67.315" x2="20.32" y2="64.915" width="0" layer="19" extent="1-1"/>
-<wire x1="20.32" y1="71.9" x2="12.065" y2="67.315" width="0" layer="19" extent="1-1"/>
-<wire x1="92.71" y1="23.81" x2="92.771" y2="44.45" width="0" layer="19" extent="1-1"/>
-<wire x1="97.155" y1="23.81" x2="92.71" y2="23.81" width="0" layer="19" extent="1-1"/>
-<wire x1="37.165" y1="5.415" x2="21.565" y2="30.315" width="0" layer="19" extent="1-1"/>
+<wire x1="29.845" y1="67.315" x2="20.32" y2="64.915" width="0" layer="19" extent="1-1"/>
+<wire x1="37.165" y1="5.415" x2="48.702" y2="31.496" width="0" layer="19" extent="1-1"/>
 </signal>
 <signal name="VCC_3V3">
@@
 <signal name="CONEX_11">
 <contactref element="U$1" pad="36"/>
+<contactref element="J2" pad="3"/>
+<wire x1="8.565" y1="5.415" x2="111.735" y2="7.375" width="0" layer="19" extent="1-1"/>
 </signal>
 <signal name="CONEX_12">
 <contactref element="U$1" pad="39"/>
+<contactref element="J2" pad="4"/>
+<wire x1="11.165" y1="5.415" x2="108.735" y2="7.375" width="0" layer="19" extent="1-1"/>
 </signal>
 <signal name="RST">
@@
 <signal name="CONEX_21">
 <contactref element="U$1" pad="34"/>
+<contactref element="J3" pad="3"/>
+<wire x1="16.365" y1="5.415" x2="123.8" y2="7.375" width="0" layer="19" extent="1-1"/>
 </signal>
 <signal name="CONEX_22">
 <contactref element="U$1" pad="35"/>
+<contactref element="J3" pad="4"/>
+<wire x1="18.965" y1="5.415" x2="120.8" y2="7.375" width="0" layer="19" extent="1-1"/>
 </signal>
 <signal name="CONEX_31">
 <contactref element="U$1" pad="25"/>
+<contactref element="J4" pad="3"/>
+<wire x1="26.765" y1="5.415" x2="135.865" y2="7.375" width="0" layer="19" extent="1-1"/>
 </signal>
 <signal name="N$13">
@@
 <signal name="CONEX_32">
 <contactref element="U$1" pad="0"/>
+<contactref element="J4" pad="4"/>
+<wire x1="18.965" y1="30.315" x2="132.865" y2="7.375" width="0" layer="19" extent="1-1"/>
 </signal>
 <signal name="N$23">
@@
 <contactref element="C7" pad="1"/>
 <contactref element="U$1" pad="5V"/>
+<contactref element="J2" pad="1"/>
+<contactref element="J3" pad="1"/>
+<contactref element="J4" pad="1"/>
+<contactref element="J5" pad="1"/>
 <wire x1="100.33" y1="50.48" x2="105.664" y2="56.007" width="0" layer="19" extent="1-1"/>
 <wire x1="97.08" y1="51.83" x2="100.33" y2="50.48" width="0" layer="19" extent="1-1"/>
-<wire x1="39.765" y1="5.415" x2="97.08" y2="51.83" width="0" layer="19" extent="1-1"/>
+<wire x1="111.735" y1="4.375" x2="100.33" y2="50.48" width="0" layer="19" extent="1-1"/>
+<wire x1="123.8" y1="4.375" x2="111.735" y2="4.375" width="0" layer="19" extent="1-1"/>
+<wire x1="135.865" y1="4.375" x2="123.8" y2="4.375" width="0" layer="19" extent="1-1"/>
+<wire x1="147.93" y1="4.375" x2="135.865" y2="4.375" width="0" layer="19" extent="1-1"/>
+<wire x1="39.765" y1="5.415" x2="111.735" y2="4.375" width="0" layer="19" extent="1-1"/>
 </signal>
 <signal name="MSHUNT_M">
@@
 <wire x1="131.76" y1="18.415" x2="136.465" y2="18.415" width="0" layer="19" extent="1-1"/>
 </signal>
-<signal name="N$9">
+<signal name="RS485_A">
 <contactref element="D1" pad="1"/>
 <contactref element="IC7" pad="6"/>
@@
 <wire x1="22.37" y1="67.8" x2="25.4" y2="64.77" width="0.3048" layer="1"/>
 <wire x1="25.4" y1="64.77" x2="28.575" y2="64.77" width="0.3048" layer="1"/>
-</signal>
-<signal name="N$14">
+<contactref element="J5" pad="3"/>
+<wire x1="28.575" y1="64.77" x2="147.93" y2="7.375" width="0" layer="19" extent="1-1"/>
+</signal>
+<signal name="RS485_B">
 <contactref element="IC7" pad="7"/>
 <contactref element="R14" pad="2"/>
@@
 <wire x1="27.94" y1="61.595" x2="31.115" y2="64.77" width="0.3048" layer="1"/>
 <wire x1="20.846" y1="61.595" x2="27.94" y2="61.595" width="0.3048" layer="1"/>
+<contactref element="J5" pad="4"/>
+<wire x1="31.115" y1="64.77" x2="144.93" y2="7.375" width="0" layer="19" extent="1-1"/>
 </signal>
 <signal name="N$3">

Commit message: coisas que fizemos durante a reuniao 18/11
Parts:
- moved D2 4.07 mm to (17.8, 59.7)
- moved D1 3.59 mm to (17.8, 67.3)
- moved RJ11_1 2.62 mm to (8.89, 62.2)
- moved RJ11_2 2.62 mm to (26.7, 62.2)
- moved C7 1.27 mm to (100.3, 50.8)
- moved C10 0.64 mm to (66.7, 33.0)
- moved C11 0.64 mm to (85.1, 44.5)
- moved C15 0.64 mm to (127.6, 19.7)
- moved R6 0.64 mm to (85.1, 48.3)
- moved R15 0.63 mm to (131.4, 18.4)
Routing:
- net GND: track 7.82 -> 0.00 mm
- net RS485_A: track 42.4 -> 39.1 mm
- net RS485_B: track 44.8 -> 47.2 mm
- net UART_RX: track 14.9 -> 13.7 mm
- net I2C_SCL: track 0.00 -> 0.94 mm
Other:
- board size 160 x 75.2 mm -> 160 x 74 mm
