File: Telemetry/2020/PCB TGE2021 v1/Projeto Principal/Versao 1_08 (eric) WIP/PCB Telemetria 2020.brd (EAGLE design)
At the start: 160 x 74 mm, 58 parts, among them IC1 INA240A1DR, IC2 MCP3221A6T-E_OTVAO, IC3 AZ1117IH-3.3TRG1, IC4 ACS758LCB-050B-PFF-T, IC5 ADS1115IDGSR, IC6 ACS712-030B3, IC7 THVD2410DR, IC8 TMP235AEDCKRQ1, J1 172042-0406, J2 43045-0412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

Commit message: WIP PCB
Parts:
- moved J5 60.9 mm to (104.8, 19.1), turned to 0 degrees
- moved J2 40.0 mm to (149.2, 15.2), turned to 270 degrees
- moved J3 33.1 mm to (144.1, 13.3), turned to 180 degrees
- moved C14 29.9 mm to (136.5, 43.2), turned to 270 degrees
- moved R11 29.6 mm to (130.8, 43.2), turned to 270 degrees
- moved IC2 26.2 mm to (130.8, 62.9), turned to 90 degrees
- moved R2 24.7 mm to (129.5, 68.6), turned to 90 degrees
- moved R1 23.8 mm to (134.6, 68.6), turned to 90 degrees
- moved C5 23.6 mm to (135.0, 58.5)
- moved U$2 21.0 mm to (114.9, 48.9), turned to 90 degrees
- moved J4 19.1 mm to (113.0, 8.26)
- moved J1 18.6 mm to (154.3, 38.7)
- moved IC6 18.1 mm to (140.3, 32.4)
- moved C3 17.6 mm to (131.2, 54.9)
- moved R3 17.3 mm to (135.0, 62.6), turned to 90 degrees
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Routing:
- net CONEX_12: track 0.00 -> 177.1 mm
- net RS485_A: track 112.8 -> 259.9 mm
- net I2C_SCL: track 4.97 -> 148.5 mm
- net I2C_SDA: track 9.56 -> 150.7 mm
- net CONEX_21: track 0.00 -> 128.1 mm
- net 12V_CM: track 5.80 -> 129.5 mm
- net CONEX_32: track 109.8 -> 0.00 mm
- net VCC_3V3: track 397.4 -> 502.4 mm
- net 12V_VM: track 14.4 -> 93.4 mm
- net VCC_5V: track 259.6 -> 184.9 mm
- net CONEX_11: track 101.9 -> 163.0 mm
- net CONEX_22: track 92.2 -> 140.6 mm
- net RS485_B: track 108.7 -> 62.5 mm
- net TEMP1: track 136.8 -> 166.3 mm
- net CMPPT_F: track 33.3 -> 3.90 mm
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