File: Telemetry/2020/PCB TGE2021 v1/Projeto Principal/Versao 1_9_roteada (agricio)/PCB Telemetria 2020.brd (EAGLE design)
At the start: 160 x 74 mm, 58 parts, among them IC1 INA240A1DR, IC2 MCP3221A6T-E_OTVAO, IC3 AZ1117IH-3.3TRG1, IC4 ACS758LCB-050B-PFF-T, IC5 ADS1115IDGSR, IC6 ACS712-030B3, IC7 THVD2410DR, IC8 TMP235AEDCKRQ1, J1 172042-0406, J2 43045-0412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

Commit message: primeira versao de roteamento - carece de revisão
Parts:
- removed J2, J3, J4, J5: 43045-0412, SamacSys_Parts:43045-0412
- added EX1, EX2, EX3: 43045-0412, SamacSys_Parts:43045-0412
- moved R9 50.2 mm to (116.2, 66.0), turned to 270 degrees
- moved C13 44.0 mm to (112.4, 64.1), turned to 180 degrees
- moved R10 42.9 mm to (112.4, 61.0), turned to 180 degrees
- moved C10 14.9 mm to (68.6, 53.6), turned to 0 degrees
- moved C18 9.71 mm to (33.0, 48.9)
- moved C12 9.69 mm to (76.2, 53.3)
- moved C7 9.09 mm to (102.2, 41.9)
- moved IC8 8.98 mm to (37.5, 48.3), turned to 0 degrees
- moved IC3 8.98 mm to (95.2, 40.6)
- moved C11 8.63 mm to (88.5, 51.1)
- moved R7 8.35 mm to (76.2, 57.9)
- moved R8 8.35 mm to (73.7, 53.3), turned to 270 degrees
- moved R6 7.30 mm to (88.5, 53.8)
- moved IC5 7.10 mm to (68.6, 50.2)
- moved C6 7.10 mm to (93.1, 35.6)
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Connections:
- removed net N$13: U$1.2
- removed net N$27: U$1.LORA2
- removed net N$28: U$1.LORA1
- removed net N$4: U$1.14
- net CONEX_11: now also EX1.1, U$1.25; no longer J2.3, U$1.36
- net CONEX_12: now also EX1.2, U$1.14; no longer J2.4, U$1.39
- net CONEX_21: now also EX2.1; no longer J3.3
- net CONEX_22: now also EX2.2; no longer J3.4
- net CONEX_31: now also EX3.1, U$1.36; no longer J4.3, U$1.25
- net CONEX_32: now also EX3.2, U$1.39; no longer J4.4, U$1.0
- net GND: now also EX1.4, EX2.4, EX3.4; no longer J2.2, J3.2, J4.2, J5.2
- net RS485_A: no longer J5.3
- net RS485_B: no longer J5.4
- net TEMP1: now also U$1.0; no longer U$1.13
- net VCC_5V: now also EX1.3, EX2.3, EX3.3; no longer J2.1, J3.1, J4.1, J5.1
Routing:
- net GND: track 257.7 -> 882.5 mm, vias 1 -> 20
- net VCC_3V3: track 0.00 -> 422.8 mm, vias 0 -> 5
- net VCC_5V: track 0.00 -> 222.3 mm, vias 0 -> 4
- net 12V_VM: track 0.00 -> 214.9 mm
- net 12V_CM: track 0.00 -> 190.8 mm
- net CONEX_31: track 0.00 -> 143.1 mm
- net CONEX_32: track 0.00 -> 137.0 mm
- net I2C_SDA: track 0.00 -> 121.7 mm
- net CONEX_21: track 0.00 -> 119.2 mm
- net I2C_SCL: track 0.00 -> 113.2 mm
- net CONEX_22: track 0.00 -> 113.1 mm
- net CONEX_11: track 0.00 -> 92.7 mm
- net CONEX_12: track 0.00 -> 86.6 mm
- net RS485_B: track 0.00 -> 43.5 mm
- net RS485_A: track 0.00 -> 39.3 mm
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- added copper zone on layer 16, net GND
