File: Telemetry/2020/PCB TGE2021 v1/Projeto Principal/Versao 1_9_roteada (agricio)/PCB Telemetria 2020.sch (EAGLE design)
At the start: 58 parts, among them IC1 INA240A1DR, IC2 MCP3221A6T-E_OTVAO, IC3 AZ1117IH-3.3TRG1, IC4 ACS758LCB-050B-PFF-T, IC5 ADS1115IDGSR, IC6 ACS712-030B3, IC7 THVD2410DR, IC8 TMP235AEDCKRQ1, J1 172042-0406, J2 43045-0412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

Commit message: primeira versao de roteamento - carece de revisão
Parts:
- removed J3, J4, J5: 43045-0412, SamacSys_Parts:43045-0412
- added EX2, EX3: 43045-0412, SamacSys_Parts:43045-0412
- renumbered J2 to EX1
Connections:
- removed net N$13: U$1.2
- removed net N$27: U$1.LORA2
- removed net N$28: U$1.LORA1
- removed net N$4: U$1.14
- net CONEX_11: now also EX1.1, U$1.25; no longer EX1.3, U$1.36
- net CONEX_12: now also EX1.2, U$1.14; no longer EX1.4, U$1.39
- net CONEX_21: now also EX2.1; no longer J3.3
- net CONEX_22: now also EX2.2; no longer J3.4
- net CONEX_31: now also EX3.1, U$1.36; no longer J4.3, U$1.25
- net CONEX_32: now also EX3.2, U$1.39; no longer J4.4, U$1.0
- net GND: now also EX1.4, EX2.4, EX3.4; no longer EX1.2, J3.2, J4.2, J5.2
- net RS485_A: no longer J5.3
- net RS485_B: no longer J5.4
- net TEMP1: now also U$1.0; no longer U$1.13
- net VCC_5V: now also EX1.3, EX2.3, EX3.3; no longer EX1.1, J3.1, J4.1, J5.1
