File: Telemetry/2020/PCB TGE2021 v1/Projeto Principal/Versao 1_09_roteada (agricio - editando)/PCB Telemetria 2020.brd (EAGLE design)
At the start: 160 x 74 mm, 57 parts, among them IC1 INA240A1DR, IC2 MCP3221A6T-E_OTVAO, IC3 AZ1117IH-3.3TRG1, IC4 ACS758LCB-050B-PFF-T, IC5 ADS1115IDGSR, IC6 ACS712-030B3, IC7 THVD2410DR, IC8 TMP235AEDCKRQ1, J1 172042-0406

Commit message: corrigindo sinais scl e sda I2C
Parts:
- moved C11 1.42 mm to (87.2, 51.7)
- moved R6 1.42 mm to (87.2, 54.5)
- moved R5 1.42 mm to (90.7, 55.5)
- moved BBANK 0.64 mm to (84.5, 64.1)
- moved VPV 0.64 mm to (69.2, 64.1)
Connections:
- removed net AIN2: IC5.6
- removed net AIN3: IC5.7
- net I2C_SCL: now also U$1.22; no longer U$1.21
- net I2C_SDA: now also U$1.21; no longer U$1.22
Routing:
- net I2C_SDA: track 121.7 -> 128.7 mm
- net GND: track 882.5 -> 879.1 mm, vias 20 -> 21
- net VCC_3V3: track 422.8 -> 424.8 mm
- net VCC_BBANK: track 7.33 -> 6.06 mm
- net I2C_SCL: track 113.2 -> 114.3 mm
- net BBANK_AIN0: track 25.7 -> 24.6 mm
