File: Telemetry/2020/PCB TGE2021 v1/Projeto Principal/Versao 1_09_roteada (agricio - editando)/PCB Telemetria 2020.sch (EAGLE design)
At the start: 57 parts, among them IC1 INA240A1DR, IC2 MCP3221A6T-E_OTVAO, IC3 AZ1117IH-3.3TRG1, IC4 ACS758LCB-050B-PFF-T, IC5 ADS1115IDGSR, IC6 ACS712-030B3, IC7 THVD2410DR, IC8 TMP235AEDCKRQ1, J1 172042-0406

Commit message: corrigindo sinais scl e sda I2C
Connections:
- removed net AIN2: IC5.AIN2
- removed net AIN3: IC5.AIN3
- net I2C_SCL: now also U$1.22; no longer U$1.21
- net I2C_SDA: now also U$1.21; no longer U$1.22
Changed lines of the file:
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@@
-</segment>
-</net>
-<net name="I2C_SDA" class="0">
-<segment>
-<pinref part="U$1" gate="G$1" pin="22"/>
-<wire x1="94.996" y1="187.96" x2="97.536" y2="187.96" width="0.1524" layer="91"/>
-<label x="97.536" y="187.96" size="1.27" layer="95" xref="yes"/>
-</segment>
-</net>
-<net name="I2C_SCL" class="0">
-<segment>
-<pinref part="U$1" gate="G$1" pin="21"/>
-<wire x1="94.996" y1="182.88" x2="97.536" y2="182.88" width="0.1524" layer="91"/>
-<label x="97.536" y="182.88" size="1.27" layer="95" xref="yes"/>
 </segment>
 </net>
@@
 <label x="97.536" y="208.28" size="1.27" layer="95" xref="yes"/>
 <pinref part="U$1" gate="G$1" pin="0"/>
+</segment>
+</net>
+<net name="I2C_SDA" class="0">
+<segment>
+<wire x1="94.996" y1="182.88" x2="97.536" y2="182.88" width="0.1524" layer="91"/>
+<label x="97.536" y="182.88" size="1.27" layer="95" xref="yes"/>
+<pinref part="U$1" gate="G$1" pin="21"/>
+</segment>
+</net>
+<net name="I2C_SCL" class="0">
+<segment>
+<wire x1="94.996" y1="187.96" x2="97.536" y2="187.96" width="0.1524" layer="91"/>
+<label x="97.536" y="187.96" size="1.27" layer="95" xref="yes"/>
+<pinref part="U$1" gate="G$1" pin="22"/>
 </segment>
 </net>
@@
 </segment>
 </net>
-<net name="AIN2" class="0">
-<segment>
-<pinref part="IC5" gate="G$1" pin="AIN2"/>
-<wire x1="68.58" y1="215.9" x2="71.12" y2="215.9" width="0.1524" layer="91"/>
-<wire x1="71.12" y1="215.9" x2="71.12" y2="208.28" width="0.1524" layer="91"/>
-<label x="71.12" y="208.28" size="1.27" layer="95" rot="R270" xref="yes"/>
-</segment>
-</net>
-<net name="AIN3" class="0">
-<segment>
-<pinref part="IC5" gate="G$1" pin="AIN3"/>
-<wire x1="68.58" y1="218.44" x2="76.2" y2="218.44" width="0.1524" layer="91"/>
-<wire x1="76.2" y1="218.44" x2="76.2" y2="208.28" width="0.1524" layer="91"/>
-<label x="76.2" y="208.28" size="1.27" layer="95" rot="R270" xref="yes"/>
-</segment>
-</net>
