File: Telemetry/2020/PCB TGE2021 v1/TGE Neil v1/eagle files/TGE NEIL v1.brd (EAGLE design)
At the start: 160 x 74 mm, 57 parts, among them IC1 INA240A1DR, IC2 MCP3221A6T-E_OTVAO, IC3 AZ1117IH-3.3TRG1, IC4 ACS758LCB-050B-PFF-T, IC5 ADS1115IDGSR, IC6 ACS712-030B3, IC7 THVD2410DR, IC8 TMP235AEDCKRQ1, J1 172042-0406

Commit message: atualizacao da versao da placa
Parts:
- moved R2 1.80 mm to (126.9, 37.2)
Connections:
- net 12V_CM: now also U$1.13; no longer U$1.33
- net 12V_VM: now also U$1.33; no longer U$1.32
- net CMPPT_F: now also U$1.32
Routing:
- net CMPPT_F: track 2.51 -> 48.0 mm
- net VCC_3V3: track 426.2 -> 385.0 mm, vias 5 -> 7
- net 12V_CM: track 191.5 -> 184.6 mm
- net 12V_VM: track 215.6 -> 212.3 mm
- net GND: track 879.9 -> 879.1 mm
Other:
- board text added: "TGE NEIL v1.0 26/08/2021"
- board text removed: "TGE NEIL v1.0 27/02/2021"
