File: Telemetry/2020/PCB TGE2021 v1/TGE Neil v1/eagle files/TGE NEIL v1.sch (EAGLE design)
At the start: 57 parts, among them IC1 INA240A1DR, IC2 MCP3221A6T-E_OTVAO, IC3 AZ1117IH-3.3TRG1, IC4 ACS758LCB-050B-PFF-T, IC5 ADS1115IDGSR, IC6 ACS712-030B3, IC7 THVD2410DR, IC8 TMP235AEDCKRQ1, J1 172042-0406

Commit message: atualizacao da versao da placa
Connections:
- net 12V_CM: now also U$1.13; no longer U$1.33
- net 12V_VM: now also U$1.33; no longer U$1.32
- net CMPPT_F: now also U$1.32
Changed lines of the file:
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@@
 <?xml version="1.0" encoding="utf-8"?>
 <!DOCTYPE eagle SYSTEM "eagle.dtd">
-<eagle version="9.5.2">
+<eagle version="9.6.2">
 <drawing>
 <settings>
@@
 <setting verticaltext="up"/>
 </settings>
-<grid distance="0.1" unitdist="inch" unit="mil" style="lines" multiple="1" display="no" altdistance="0.01" altunitdist="inch" altunit="inch"/>
+<grid distance="0.1" unitdist="inch" unit="inch" style="lines" multiple="1" display="no" altdistance="0.01" altunitdist="inch" altunit="inch"/>
 <layers>
 <layer number="1" name="Top" color="4" fill="1" visible="no" active="no"/>
@@
 </segment>
 </net>
-<net name="12V_CM" class="0">
-<segment>
-<pinref part="U$1" gate="G$1" pin="33"/>
-<wire x1="51.816" y1="198.12" x2="49.276" y2="198.12" width="0.1524" layer="91"/>
-<label x="49.276" y="198.12" size="1.27" layer="95" rot="R180" xref="yes"/>
-</segment>
-</net>
 <net name="GND" class="0">
 <segment>
@@
 </segment>
 </net>
-<net name="12V_VM" class="0">
-<segment>
-<pinref part="U$1" gate="G$1" pin="32"/>
-<wire x1="51.816" y1="203.2" x2="49.276" y2="203.2" width="0.1524" layer="91"/>
-<label x="49.276" y="203.2" size="1.27" layer="95" rot="R180" xref="yes"/>
-</segment>
-</net>
 <net name="CONEX_12" class="0">
 <segment>
@@
 </segment>
 </net>
+<net name="12V_VM" class="0">
+<segment>
+<wire x1="51.816" y1="198.12" x2="49.276" y2="198.12" width="0.1524" layer="91"/>
+<label x="49.276" y="198.12" size="1.27" layer="95" rot="R180" xref="yes"/>
+<pinref part="U$1" gate="G$1" pin="33"/>
+</segment>
+</net>
+<net name="CMPPT_F" class="0">
+<segment>
+<pinref part="U$1" gate="G$1" pin="32"/>
+<wire x1="51.816" y1="203.2" x2="48.26" y2="203.2" width="0.1524" layer="91"/>
+<label x="48.26" y="203.2" size="1.27" layer="95" rot="R180" xref="yes"/>
+</segment>
+</net>
+<net name="12V_CM" class="0">
+<segment>
+<wire x1="51.816" y1="182.88" x2="49.276" y2="182.88" width="0.1524" layer="91"/>
+<label x="49.276" y="182.88" size="1.27" layer="95" rot="R180" xref="yes"/>
+<pinref part="U$1" gate="G$1" pin="13"/>
+</segment>
+</net>
